File: hybrid-tube-amp.kicad_sch (KiCad schematic)
At the start: 0 parts

Commit message: Updated schematic up to but not including BOM and footprint assignment
Parts:
- added D101: 1N4148, symbol Device:D
- added J101, J102: 282834-2, symbol Connector:Screw_Terminal_01x02
- added J103, J104: 1711725, symbol Connector:Screw_Terminal_01x02
- added K101: RT424012F, symbol Relay:Relay_DPDT
- added L101, L102: 2u, symbol Device:L
- added R101, R102: 10, symbol Device:R_US
- added R103: 180, symbol Device:R_US
Connections:
- new net: K101.14, L102.2, R102.2
- new net: J104.1 (Pin_1), K101.11
- new net: J103.1 (Pin_1), K101.21
- new net: K101.24, L101.2, R101.2
- new net: D101.2 (A), K101.A1, R103.1
- new net +18V: D101.1 (K), K101.A2
- new net Auxiliaries/DELAY_RDY: R103.2
- new net GND: J101.2 (Pin_2), J102.2 (Pin_2), J103.2 (Pin_2), J104.2 (Pin_2), K101.12, K101.22
- new net Input amp/IN_L: J101.1 (Pin_1)
- new net Input amp/IN_R: J102.1 (Pin_1)
- new net Left Channel/OUT: L101.1, R101.1
- new net Right Channel/OUT: L102.1, R102.1
Other:
- added sheet Auxiliaries (aux.kicad_sch)
- added sheet Input amp (input_amp.kicad_sch)
- added sheet Left Channel (main_amp.kicad_sch)
- added sheet Power (power.kicad_sch)
- added sheet Right Channel (main_amp.kicad_sch)
- note added: "Auxiliary (off-board) parts: Connex SMPS300REh: Power supply. Neutrik NF2D-B-9: RCA jack (white) x3 (Audio inputs) Neutrik NF2D-B-2: RCA jack (red) x3 (Audio inputs) Mueller Electric BU-P3770-0 (black) x2 (Speaker post) Mueller Electric BU-P3770-2 (red) x2 (Speaker post) PIHER PC16IP04103A (10k potentiometer) (balance control) Omeg PO4S-LIN 100K (100k potentiometer) (Volume control) Schurter 4304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"
- note added: "Hand-wound output inductors. Care with layout not to have them interfere."
- note added: "Input connectors"
- note added: "Mechanical parts list: 1x Wakefield 120-2 (Thermal paste) 8x Aavid 4180G (Al2O3 insulators, TO-3P, for output devices, 4 per channel) 10x Aavid 4171G (Al2O3 insulators, TO-220, for drivers and bias generator, 5 per channel) 18x Bivar SW‑185‑150 (insulating washer for screw holes, M3 screw, needed for all heatsinked transistors) 18x M3 flat washer, stainless steel 18x M3 spring-lock washer, stainl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"
- note added: "Speaker connectors"
- title: (none) -> 100W Hybrid Audio Amplifier

Commit message: Completed schematic
Parts:
- added D? (x4): D, symbol Device:D
Connections:
- net at J104.1 (Pin_1), K101.11: now also D?.1 (K), D?.2 (A)
- net at J103.1 (Pin_1), K101.21: now also D?.1 (K), D?.2 (A)
- new net +30V: D?.1 (K), D?.1 (K)
- new net -30V: D?.2 (A), D?.2 (A)
Other:
- sheet Auxiliaries ports: added CH_L, CH_R, DC_FAULT; removed none
- moved on the sheet: D101, K101, L101, L102, R101, R102, R103
