File: main_amp.kicad_sch (KiCad schematic)
At the start: 65 parts, among them Q201 KSA992, Q202 KSC1845, Q203 KSC1845, Q204 KSC1845, Q205 KSA992, Q206 KSC1845, Q207 KSC1845, Q208 BD140, Q209 BD140, Q210 KSC1845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

Commit message: Completed schematic
Parts:
- removed C202: 4.7u, symbol Device:C_Polarized
- removed R210: 50k, symbol Device:R_US
- added C202: 4.7u, Capacitor_THT:C_Disc_D5.0mm_W2.5mm_P2.50mm, symbol Device:C
- added D202, D203, D204: 1N4148, symbol Device:D
- C201: footprint (none) -> Capacitor_THT:CP_Radial_D8.0mm_P3.50mm; MPN (none) -> UPW1J470MPD; Orderable Part Number (none) -> 647-UPW1J470MPD
- C204: value 220p -> 100p; footprint (none) -> Capacitor_SMD:C_0603_1608Metric_Pad1.08x0.95mm_HandSolder; MPN (none) -> C0603C101J1GACTU; Orderable Part Number (none) -> 80-C0603C101J1G
- C205: MPN (none) -> UKA1V102MHD; Orderable part number (none) -> 647-UKA1V102MHD
- R201: value 50k -> 22k
- R234: value 1.2k -> 100
- R235: value 22k -> 2.2k
Connections:
- net GND: now also D203.1 (K), D204.2 (A); no longer D201.2 (A)
- net cathode_common: now also C202.1
- net at C205.1, D201.1 (K), R234.1: now also D202.2 (A)
- net at Q202.3 (B), Q206.3 (B), R211.2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: now also C202.2
- new net: D202.1 (K), D203.2 (A)
- new net: D201.2 (A), D204.1 (K)
Other:
- moved on the sheet: D201
