File: power.kicad_sch (KiCad schematic)
At the start: 35 parts, among them J501 TB009-508-05BE, U501 MC34063AP, U502 LM317_TO-220, U503 LM337_TO220, U504 LM7812_TO220

Commit message: Completed schematic
Parts:
- removed C511, C512, C514, C515: 1000u, symbol Device:C_Polarized
Other:
- moved on the sheet: J501
